File: hw/picocart64_v1/Concept2.kicad_sch (KiCad schematic)
At the start: 10 parts

Commit message: hw: Add power budget, updated BOM
Parts:
- J?: value (none) -> Conn_02x06_Odd_Even; footprint (none) -> Connector_PinSocket_2.54mm:PinSocket_2x06_P2.54mm_Horizontal
- J?: value (none) -> Micro_SD_Card_Det; footprint (none) -> Connector_Card:microSD_HC_Molex_104031-0811
- J?: value (none) -> Conn_01x05; footprint (none) -> Connector_PinHeader_2.54mm:PinHeader_1x05_P2.54mm_Vertical
- JP? (x4): value (none) -> SolderJumper_2_Open; footprint (none) -> Jumper:SolderJumper-2_P1.3mm_Open_TrianglePad1.0x1.5mm
- SW?: value (none) -> BootButton; footprint (none) -> Button_Switch_SMD:SW_SPST_FSMSM
- U?: value (none) -> N64-Cartridge; footprint (none) -> picocart64:N64-Connector
- U?: value (none) -> RP2040_Stamp; footprint (none) -> RP2040_Stamp:RP2040_Stamp_FlexyPin
Other:
- note added: "BOM: @ qty 1 (will be cheaper when producing 100x +) 2x RP2040 = $2 WiFi Module (ESP32) = $3 MC74AC138 = $1 SDCard slot = $0.5 4 x LY68L6400SLIT = $11 USB conn. = $0.5 SPI Flash (16MB) = $1.1 W25Q128JVSIQ SPI Flash (2MB) = $0.5 W25Q16JVSSIQ 2 x Crystal 12MHz = $0.5 XYDBPCNANF-12MHZ / C521567 5V -> 3.3V 1A LDO = $0.34 SSP1117-3.3V / C277892 TBD 5V/3.3V switch = $1 BSS84 is too weak PCB = $1 Total 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"
- note added: "POWER BUDGET 2x RP2040 2*100(?) = 200mA (let's use max rating @133MHz) 8x PSRAM ly68l6400slit 1 * 40 = 40mA (only draws I during read/write) 8 * 1 = 8mA (idle current) 1x ESP32 345 mA (!) during wifi tx 1x SDCard (SPI mode) 150mA Total: 200+40+8+345+150 = 743 mA Need _at least_ 750mA supply, 1A recommended."
- note removed: "BOM: @ qty 1 (will be cheaper when producing 100x +) 2x RP2040 = $2 WiFi Module (ESP32) = $3 MC74AC138 = $1 SDCard slot = $0.5 4 x LY68L6400SLIT = $11 USB conn. = $0.5 SPI Flash (16MB) = $1.1 W25Q128JVSIQ SPI Flash (2MB) = $0.5 W25Q16JVSSIQ 2 x Crystal 12MHz = $0.5 XYDBPCNANF-12MHZ / C521567 PCB = $1 Total 2+3+1+0.5+11+0.5+1.1+0.5+0.5+1 = $21.1 Customer price = 3 * BOM = $63.3"
