File: hw/picocart64_v1/Concept1.kicad_sch (KiCad schematic)
At the start: 10 parts

Commit message: hw: Concept3
Parts:
- removed J?: Conn_02x06_Odd_Even, Connector_PinSocket_2.54mm:PinSocket_2x06_P2.54mm_Horizontal, symbol Connector_Generic:Conn_02x06_Odd_Even
- removed J?: Micro_SD_Card_Det, Connector_Card:microSD_HC_Molex_104031-0811, symbol Connector:Micro_SD_Card_Det
- removed J?: Conn_01x05, Connector_PinHeader_2.54mm:PinHeader_1x05_P2.54mm_Vertical, symbol Connector_Generic:Conn_01x05
- removed JP? (x4): SolderJumper_2_Open, Jumper:SolderJumper-2_P1.3mm_Open_TrianglePad1.0x1.5mm, symbol Jumper:SolderJumper_2_Open
- removed SW?: BootButton, Button_Switch_SMD:SW_SPST_FSMSM, symbol Switch:SW_Push
- removed U?: N64-Cartridge, picocart64:N64-Connector, symbol n64-cartridge:N64-Cartridge
- removed U?: RP2040_Stamp, RP2040_Stamp:RP2040_Stamp_FlexyPin, symbol RP2040_Stamp:RP2040_Stamp
- added J?: Conn_01x05, Connector_PinHeader_2.54mm:PinHeader_1x05_P2.54mm_Vertical, symbol Connector_Generic:Conn_01x05
- added J?: Micro_SD_Card_Det, Connector_Card:microSD_HC_Molex_104031-0811, symbol Connector:Micro_SD_Card_Det
- added J?: Conn_02x06_Odd_Even, Connector_PinSocket_2.54mm:PinSocket_2x06_P2.54mm_Horizontal, symbol Connector_Generic:Conn_02x06_Odd_Even
- added JP? (x4): SolderJumper_2_Open, Jumper:SolderJumper-2_P1.3mm_Open_TrianglePad1.0x1.5mm, symbol Jumper:SolderJumper_2_Open
- added SW?: BootButton, Button_Switch_SMD:SW_SPST_FSMSM, symbol Switch:SW_Push
- added U?: RP2040_Stamp, RP2040_Stamp:RP2040_Stamp_FlexyPin, symbol RP2040_Stamp:RP2040_Stamp
- added U?: N64-Cartridge, picocart64:N64-Connector, symbol n64-cartridge:N64-Cartridge
Connections:
- net +3V3: now also J?.1 (Pin_1), J?.1 (Pin_1), J?.2 (Pin_2), J?.4 (VDD), U?.34 (3.3V)
- net AD0: now also U?.1 (GPIO0), U?.28 (AD0)
- net AD1: now also U?.2 (GPIO1), U?.29 (AD1)
- net AD10: now also U?.11 (GPIO10), U?.12 (AD10)
- net AD11: now also U?.11 (AD11), U?.12 (GPIO11)
- net AD12: now also U?.13 (GPIO12), U?.7 (AD12)
- net AD13: now also U?.14 (GPIO13), U?.5 (AD13)
- net AD14: now also U?.15 (GPIO14), U?.4 (AD14)
- net AD15: now also U?.16 (GPIO15), U?.3 (AD15)
- net AD2: now also U?.3 (GPIO2), U?.30 (AD2)
- net AD3: now also U?.32 (AD3), U?.4 (GPIO3)
- net AD4: now also U?.36 (AD4), U?.5 (GPIO4)
- net AD5: now also U?.37 (AD5), U?.6 (GPIO5)
- net AD6: now also U?.40 (AD6), U?.7 (GPIO6)
- net AD7: now also U?.41 (AD7), U?.8 (GPIO7)
- net AD8: now also U?.16 (AD8), U?.9 (GPIO8)
- net AD9: now also U?.10 (GPIO9), U?.15 (AD9)
- net ALEH: now also U?.18 (GPIO17), U?.35 (aleH)
- net ALEL: now also U?.17 (GPIO16), U?.33 (aleL)
- net GND: now also J?.11 (SHIELD), J?.3 (Pin_3), J?.4 (Pin_4), J?.5 (Pin_5), J?.6 (VSS), J?.9 (DET_B), SW?.1, U?.1 (GND), U?.2 (GND), U?.22 (GND), U?.23 (GND), U?.25 (GND), U?.26 (GND), U?.27 (GND), U?.31 (GND), U?.31 (GND), U?.47 (GND), U?.48 (GND), U?.50 (GND), U?.6 (GND)
- net N64_CIC_DCLK: now also U?.21 (GPIO20), U?.43 (u3_14)
- net N64_CIC_DIO: now also U?.18 (u3_15), U?.22 (GPIO21)
- net N64_COLD_RESET: now also U?.20 (COLD_RESET), U?.23 (GPIO22)
- net N64_EEP_SDAT: now also JP?.2 (B)
- net N64_INT: now also JP?.2 (B), U?.44 (NC)
- net N64_NMI: now also U?.45 (os_event_cart)
- net N64_SI_CLK: now also JP?.2 (B), U?.19 (1.6mHz)
- net N64_S_DAT: now also JP?.2 (B), U?.21 (S_DAT)
- net N64_VCC: now also U?.17 (VCC), U?.34 (VCC), U?.42 (VCC), U?.9 (VCC)
- net PMOD_1_SS: now also J?.11 (Pin_11), J?.3 (CMD), JP?.1 (A), U?.26 (GPIO25)
- net PMOD_2_SIO0: now also J?.7 (DAT0), J?.9 (Pin_9), U?.28 (GPIO27)
- net PMOD_3_SIO1: now also J?.7 (Pin_7), J?.8 (DAT1), U?.29 (GPIO28)
- net PMOD_4_SCLK: now also J?.5 (CLK), J?.5 (Pin_5), JP?.1 (A), U?.27 (GPIO26)
- net PMOD_5_SIO2: now also J?.1 (DAT2), J?.12 (Pin_12), JP?.1 (A), U?.24 (GPIO23)
- net PMOD_6_SIO3: now also J?.10 (Pin_10), J?.2 (DAT3/CD), JP?.1 (A), U?.25 (GPIO24)
- net PMOD_7_CS0: now also J?.10 (DET_A), J?.8 (Pin_8), U?.30 (GPIO29)
- net PMOD_8_CS1: now also J?.6 (Pin_6)
- net RP_SWDCLK: now also J?.3 (Pin_3), U?.38 (SWCLK)
- net RP_SWDIO: now also J?.4 (Pin_4), U?.37 (SWDIO)
- net USB_D+: now also U?.36 (USB_D+)
- net USB_D-: now also U?.35 (USB_D-)
- net VBUS: now also U?.33 (5V)
- net ~{READ}: now also U?.10 (READ), U?.20 (GPIO19)
- net ~{RP_RESET}: now also J?.2 (Pin_2), U?.39 (~{RESET})
- net ~{WRITE}: now also U?.19 (GPIO18), U?.8 (WRITE)
- new net: SW?.2, U?.40 (BOOTSEL)
