File: hw/picocart64_v1/Concept3.kicad_sch (KiCad schematic)
At the start: 10 parts

Commit message: hw: Update Concept3
Parts:
- J?: value (none) -> Conn_02x06_Odd_Even; footprint (none) -> Connector_PinSocket_2.54mm:PinSocket_2x06_P2.54mm_Horizontal
- J?: value (none) -> Micro_SD_Card_Det; footprint (none) -> Connector_Card:microSD_HC_Molex_104031-0811
- J?: value (none) -> Conn_01x05; footprint (none) -> Connector_PinHeader_2.54mm:PinHeader_1x05_P2.54mm_Vertical
- JP? (x4): value (none) -> SolderJumper_2_Open; footprint (none) -> Jumper:SolderJumper-2_P1.3mm_Open_TrianglePad1.0x1.5mm
- SW?: value (none) -> BootButton; footprint (none) -> Button_Switch_SMD:SW_SPST_FSMSM
- U?: value (none) -> N64-Cartridge; footprint (none) -> picocart64:N64-Connector
- U?: value (none) -> RP2040_Stamp; footprint (none) -> RP2040_Stamp:RP2040_Stamp_FlexyPin
Other:
- note added: "EN"
- note added: "Pico2 Pin Count = 5+3+1+1+1+1+2+6+5+1+4 = 30"
- note added: "SPI Boot Mode"
- note added: "Wifi Module, ESP32-C3"
- note removed: "4 free IO"
- note removed: "Pico2 Pin Count = 5+3+1+1+1+1+2+5+3+4 = 26"
- note removed: "UART + Boot"
- note removed: "Wifi Module"
