File: hw/picocart64_v2/board.kicad_sch (KiCad schematic)
At the start: 81 parts, among them J1 USB_C_Receptacle_USB2.0, J2 USB_C_Receptacle_USB2.0, J3 Conn_02x06_Odd_Even, J4 Micro_SD_Card_Det, J5 Conn_01x02, J6 Conn_01x06, Q1 FDN340P, SW1 BootButton, U10 USBLC6-2SC6, U11 AZ1117-3.3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

Commit message: Updated schematic for larger resistor arrays, removed the extra flash chip and only use the existing 8 pads, it will default to 1 for booting/loading firmware. Added a reset button to the back. Added company logo and updated text on board.
Parts:
- removed C39: 100n, Capacitor_SMD:C_0402_1005Metric, symbol Device:C_Small
- removed R7: 10K, Resistor_SMD:R_0402_1005Metric, symbol Device:R_Small
- removed U13: W25Q128JVS, Package_SO:SOIC-8_5.23x5.23mm_P1.27mm, symbol Memory_Flash:W25Q128JVS
- added SW2: ResetButton, Button_Switch_SMD:SW_SPST_FSMSM, symbol Switch:SW_Push
- RN1, RN2, RN3, RN4, RN5, RN6: footprint Resistor_SMD:R_Array_Convex_4x0402 -> Resistor_SMD:R_Array_Convex_4x0603
Connections:
- net GND: now also SW2.2
- net MCU2_RUN: now also SW2.1
Other:
- note added: "Reset"
- note removed: "NOTE: May switch to smaller flash later. Let's go for 16MB, makes it easier to develop."
